File: Hardware/PCB_Nelven/ChaSouRo/ChaSouRo.kicad_pcb (KiCad board)
At the start: 4 copper layers, 57 x 54 mm, 91 parts, among them IC1 ADXL343BCCZ-RL, IC2 ZXBM5210-SP-13, IC3 MP1475DJ-LF-P, IC4 ZXBM5210-SP-13, IC5 BU33SD5WG-TR, J1 LiDAR, J10 Motor_R, J11 BATT, J12 Buzz, J2 OLED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

Commit message: maj PCB
Parts:
- added C32: 0.1u, Capacitor_SMD:C_0402_1005Metric, B.Cu at (147.5, 80.4)
- added C33: 0.1u, Capacitor_SMD:C_0402_1005Metric, B.Cu at (147.0, 91.0)
- added C34: 0.1u, Capacitor_SMD:C_0402_1005Metric, B.Cu at (108.1, 90.6)
- added C35: 0.1u, Capacitor_SMD:C_0402_1005Metric, B.Cu at (107.9, 80.6)
Routing:
- net OUT_1_L: track 0.00 -> 2.04 mm
- net /Power&Control/OUT_2_L: track 0.00 -> 2.01 mm
- net OUT_1_R: track 0.00 -> 1.87 mm
- net /Power&Control/OUT_2_R: track 0.00 -> 1.67 mm
- net GND: vias 58 -> 110
