File: Hardware/PCB_Nelven/ChaSouRo/Power&Control.kicad_sch (KiCad schematic)
At the start: 34 parts, among them IC2 ZXBM5210-SP-13, IC3 MP1475DJ-LF-P, IC4 ZXBM5210-SP-13, IC5 BU33SD5WG-TR, J10 Motor_R, J11 BATT, J9 Motor_L

Commit message: maj PCB
Parts:
- added C32, C33, C34, C35: 0.1u, Capacitor_SMD:C_0402_1005Metric, symbol Device:C_Small
Connections:
- net GND: now also C32.2, C33.2, C34.2, C35.2
- net OUT_1_L: now also C32.1
- net OUT_1_R: now also C34.1
- net OUT_2_L: now also C33.1
- net OUT_2_R: now also C35.1
