File: Hardware/ChaSouRo/sensors&periphs.kicad_sch (KiCad schematic)
At the start: 18 parts, among them IC1 ADXL343BCCZ-RL, J1 LiDAR, J12 Buzz, J2 OLED, J4 BT, J5 ToF1, J6 ToF2, J7 ToF3, J8 ToF4, Q1 IRLML2060

Commit message: maj PCB
Other:
- note removed: "2502 si possible"
Changed lines of the file:
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@@
-		)
-	)
-	(text "2502 si possible"
-		(exclude_from_sim no)
-		(at 213.106 95.25 0)
-		(effects
-			(font
-				(size 1.27 1.27)
-			)
 		)
 	)
