File: Hardware/ChaSouRo/Power&Control.kicad_sch (KiCad schematic)
At the start: 38 parts, among them IC2 ZXBM5210-SP-13, IC3 MP1475DJ-LF-P, IC4 ZXBM5210-SP-13, IC5 BU33SD5WG-TR, J10 Motor_R, J11 BATT, J9 Motor_L

Commit message: maj PCB
Parts:
- IC3: footprint ESE:SOT65P280X100-8N -> Package_TO_SOT_SMD:TSOT-23-8
Changed lines of the file:
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@@
 			)
 		)
-		(property "Footprint" "ESE:SOT65P280X100-8N"
+		(property "Footprint" "Package_TO_SOT_SMD:TSOT-23-8"
 			(at 194.31 135.56 0)
 			(effects
@@
 				)
 				(justify left top)
-				(hide yes)
 			)
 		)
