File: Hardware/ChaSouRo/ChaSouRo.kicad_pcb (KiCad board)
At the start: 4 copper layers, 57 x 54 mm, 95 parts, among them IC1 ADXL343BCCZ-RL, IC2 ZXBM5210-SP-13, IC3 MP1475DJ-LF-P, IC4 ZXBM5210-SP-13, IC5 BU33SD5WG-TR, J1 LiDAR, J10 Motor_R, J11 BATT, J12 Buzz, J2 OLED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

Commit message: maj PCB
Connections:
- C8 pad 1: /VREF+ -> +3.3V
- C9 pad 1: /VREF+ -> +3.3V
- U1 pad 20: /VREF+ -> +3.3V
Routing:
- net /VREF+: track 2.04 -> 0.00 mm, vias 1 -> 0
- net +3.3V: track 27.8 -> 29.8 mm, vias 15 -> 16
- net ENC_PA_R: track 25.3 -> 26.0 mm
- net ENC_PB_R: track 27.9 -> 28.5 mm

Commit message: maj PCB
Parts:
- D1: value 1 -> D1
- D2: value 2 -> D2
- IC3: footprint ESE:SOT65P280X100-8N -> Package_TO_SOT_SMD:TSOT-23-8
- moved G*** 0.60 mm to (114.0, 62.5)
Other:
- board text added: "+"
- board text added: "-"
- board text added: "3.3V"
- board text added: "5V"
- board text added: "Batt"
- board text added: "Buzz"
- board text added: "CTRL"
- board text added: "EN"
- board text added: "GND"
- board text added: "IN"
- board text added: "Out1"
- board text added: "Out2"
- board text added: "PA"
- board text added: "PB"
- board text added: "RX2"
- board text added: "RX3"
- board text added: "SCL1"
- board text added: "SCL3"
- board text added: "SDA1"
- board text added: "SDA3"
- board text added: "TX3"
- board text added: "XSt1"
- board text added: "XSt2"
- board text added: "XSt3"
- board text added: "XSt4"

Commit message: check pcb LF
Parts:
- D1: value D1 -> 1
- D2: value D2 -> 2
Connections:
- J3 pad 13: TX4 -> RX4
- J3 pad 14: RX4 -> TX4
Routing:
- net RX4: track 10.6 -> 14.8 mm, vias 0 -> 2
- net TX4: track 13.6 -> 10.1 mm, vias 2 -> 0
- net +5V: track 40.8 -> 38.7 mm
- added copper zone on B.Cu, net +5V

Commit message: ajout d'un SW PCB
Parts:
- S2: value USER -> USER1
Connections:
- net /USER renamed /USER1
- U1 pad 9: unconnected-(U1-PA1-Pad9) -> USER2
Routing:
- net USER2: track 0.00 -> 32.8 mm, vias 0 -> 1
- net TX2: track 3.30 -> 2.80 mm
- net GND: vias 110 -> 111
Other:
- board text added: "USER2"
