File: Hardware/ChaSouRo/ChaSouRo.kicad_sch (KiCad schematic)
At the start: 38 parts, among them J3 Conn_ST_STDC14, U1 STM32G431CBUx, Y1 Crystal_GND24_Small

Commit message: maj PCB
Connections:
- net VREF+ is gone; now on net +3.3V: C8.1, C9.1, U1.20 (VREF+)
Changed lines of the file:
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@@
+	)
+	(junction
+		(at 170.18 50.8)
+		(diameter 0)
+		(color 0 0 0 0)
 	)
 	(junction
@@
 					(unit 1)
 				)
+			)
+		)
+	)
+	(symbol
+		(lib_id "power:+3.3V")
+		(at 170.18 50.8 0)
+		(unit 1)
+		(exclude_from_sim no)
+		(in_bom yes)
+		(on_board yes)
+		(dnp no)
+		(fields_autoplaced yes)
+		(property "Reference" "#PWR017"
+			(at 170.18 54.61 0)
+			(effects
+				(font
+					(size 1.27 1.27)
+				)
+				(hide yes)
+			)
+		)
+		(property "Value" "+3.3V"
+			(at 170.18 45.72 0)
+			(effects
+				(font
+					(size 1.27 1.27)
+				)
+			)
+		)
+		(property "Footprint" ""
+			(at 170.18 50.8 0)
+			(effects
+				(font
+					(size 1.27 1.27)
+				)
+				(hide yes)
+			)
+		)
+		(property "Datasheet" ""
+			(at 170.18 50.8 0)
+			(effects
+				(font
+					(size 1.27 1.27)
+				)
+				(hide yes)
+			)
+		)
+		(property "Description" "Power symbol creates a global label with name \"+3.3V\""
+			(at 170.18 50.8 0)
+			(effects
+				(font
+					(size 1.27 1.27)
+				)
+				(hide yes)
+			)
+		)
+		(pin "1"
+		)
+		(instances
+			(project "ChaSouRo"
+				(path "/831bd0a7-ff0c-4dec-8880-0dfe5b65c90c"
+					(reference "#PWR017")
+					(unit 1)
+				)

Commit message: check pcb LF
Connections:
- net RX4: now also J3.13 (VCP_RX); no longer J3.14 (VCP_TX)
- net TX4: now also J3.14 (VCP_TX); no longer J3.13 (VCP_RX)
Changed lines of the file:
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@@
 	(global_label "RX4"
 		(shape input)
-		(at 270.51 129.54 0)
+		(at 270.51 127 0)
 		(fields_autoplaced yes)
 		(effects
@@
 		)
 		(property "Intersheetrefs" "${INTERSHEET_REFS}"
-			(at 277.6602 129.54 0)
+			(at 277.6602 127 0)
 			(effects
 				(font
@@
 	(global_label "TX4"
 		(shape input)
-		(at 270.51 127 0)
+		(at 270.51 129.54 0)
 		(fields_autoplaced yes)
 		(effects
@@
 		)
 		(property "Intersheetrefs" "${INTERSHEET_REFS}"
-			(at 277.3578 127 0)
-			(effects
-				(font
+			(at 277.3578 129.54 0)
+			(effects
+				(font

Commit message: ajout d'un SW PCB
Parts:
- added TP8: USER2, symbol Connector:TestPoint
Connections:
- net USER2: now reaches U1.9 (PA1)
- net USER2: now also TP8.1
- net USER renamed USER1
- no-connect marks 9 -> 8
Changed lines of the file:
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@@
 	)
 	(no_connect
-		(at 231.14 57.15)
-	)
-	(no_connect
 		(at 270.51 116.84)
 	)
@@
 		)
 	)
-	(label "USER"
+	(label "USER1"
 		(at 166.37 115.57 0)
 		(effects
@@
 		)
 	)
-	(label "VREF+"
-		(at 189.23 50.8 0)
-		(effects
-			(font
-				(size 1.27 1.27)
-			)
-			(justify left bottom)
-		)
-	)
 	(label "D1"
 		(at 179.07 101.6 0)
@@
 		)
 	)
+	(global_label "USER2"
+		(shape input)
+		(at 231.14 57.15 0)
+		(fields_autoplaced yes)
+		(effects
+			(font
+				(size 1.27 1.27)
+			)
+			(justify left)
+		)
+		(property "Intersheetrefs" "${INTERSHEET_REFS}"
+			(at 240.2937 57.15 0)
+			(effects
+				(font
+					(size 1.27 1.27)
+				)
+				(justify left)
+				(hide yes)
+			)
+		)
+	)
 	(global_label "SWDIO"
 		(shape input)
@@
 		)
 	)
+	(global_label "USER2"
+		(shape input)
+		(at 45.72 181.61 270)
+		(fields_autoplaced yes)
+		(effects
+			(font
+				(size 1.27 1.27)
+			)
+			(justify right)
+		)
+		(property "Intersheetrefs" "${INTERSHEET_REFS}"
+			(at 45.72 190.7637 90)
+			(effects
+				(font
+					(size 1.27 1.27)
+				)
+				(justify right)
+				(hide yes)
+			)
+		)
+	)
 	(global_label "ENC_PA_R"
 		(shape input)
@@
 					(unit 1)
 				)
+			)
+		)
+	)
+	(symbol
+		(lib_id "Connector:TestPoint")
+		(at 45.72 181.61 0)
+		(unit 1)
+		(exclude_from_sim no)
+		(in_bom yes)
+		(on_board yes)
+		(dnp no)
+		(property "Reference" "TP8"
+			(at 51.308 179.578 0)
+			(effects
+				(font
+					(size 1.27 1.27)
+				)
+				(justify right)
+			)
+		)
+		(property "Value" "USER2"
+			(at 51.308 176.784 0)
+			(effects
+				(font
+					(size 1.27 1.27)
+				)
+				(justify right)
+			)
+		)
+		(property "Footprint" ""
+			(at 50.8 181.61 0)
+			(effects
+				(font
+					(size 1.27 1.27)
+				)
+				(hide yes)
+			)
+		)
+		(property "Datasheet" "~"
+			(at 50.8 181.61 0)
+			(effects
+				(font
+					(size 1.27 1.27)
+				)
+				(hide yes)
+			)
+		)
+		(property "Description" "test point"
+			(at 45.72 181.61 0)
+			(effects
+				(font
+					(size 1.27 1.27)
+				)
+				(hide yes)
+			)
+		)
+		(pin "1"
+		)
+		(instances
+			(project "ChaSouRo"
+				(path "/831bd0a7-ff0c-4dec-8880-0dfe5b65c90c"
+					(reference "TP8")
+					(unit 1)
+				)
