File: Hardware/V2/ChaSouRo/ChaSouRo.kicad_pcb (KiCad board)
At the start: 4 copper layers, 57 x 54 mm, 96 parts, among them IC1 ADXL343BCCZ-RL, IC2 ZXBM5210-SP-13, IC3 MP1475DJ-LF-P, IC4 ZXBM5210-SP-13, IC5 BU33SD5WG-TR, J1 LiDAR, J10 Motor_R, J11 BATT + ON/OFF, J12 Buzz, J2 OLED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

Commit message: modif pcb
Parts:
- moved G*** 8.01 mm to (112.7, 70.5)
- moved TP3 7.53 mm to (115.0, 63.4), turned to 180 degrees
- moved TP2 3.41 mm to (116.3, 71.0)
Changed lines of the file:
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@@
 	(footprint "TestPoint:TestPoint_Bridge_Pitch2.0mm_Drill0.7mm"
 		(layer "F.Cu")
-		(at 116.7 70.7 90)
+		(at 115.05 63.35 180)
 		(descr "wire loop as test point, pitch 2.0mm, hole diameter 0.7mm, wire diameter 0.5mm")
 		(tags "test point wire loop")
 		(property "Reference" "TP3"
-			(at 1.1 1.7 90)
+			(at 1.1 1.7 0)
 			(layer "F.SilkS")
 			(hide yes)
@@
 		)
 		(property "Value" "3V3"
-			(at -1.8 0 0)
+			(at 1 1.65 180)
 			(unlocked yes)
 			(layer "F.SilkS")
@@
 		)
 		(property "Datasheet" ""
-			(at 0 0 90)
+			(at 0 0 180)
 			(unlocked yes)
 			(layer "F.Fab")
@@
 		)
 		(property "Description" "test point"
-			(at 0 0 90)
+			(at 0 0 180)
 			(unlocked yes)
 			(layer "F.Fab")
@@
 		(attr through_hole)
 		(fp_line
-			(start 2.9 -0.9)
-			(end -0.9 -0.9)
+			(start 2.9 0.9)
+			(end 2.9 -0.9)
 			(stroke
 				(width 0.12)
@@
 		)
 		(fp_line
-			(start -0.9 -0.9)
-			(end -0.9 0.9)
+			(start 2.9 -0.9)
+			(end -0.9 -0.9)
 			(stroke
 				(width 0.12)
@@
 		)
 		(fp_line
-			(start 2.9 0.9)
-			(end 2.9 -0.9)
+			(start -0.9 0.9)
+			(end 2.9 0.9)
 			(stroke
 				(width 0.12)
@@
 		)
 		(fp_line
-			(start -0.9 0.9)
-			(end 2.9 0.9)
+			(start -0.9 -0.9)
+			(end -0.9 0.9)
 			(stroke
 				(width 0.12)
@@
 		(fp_line
 			(start 3.2 -1.2)
-			(end -1.2 -1.2)
+			(end 3.2 1.2)
 			(stroke
 				(width 0.05)
@@
 		(fp_line
 			(start 3.2 -1.2)
-			(end 3.2 1.2)
+			(end -1.2 -1.2)
 			(stroke
 				(width 0.05)
@@
 		(fp_line
 			(start -1.2 1.2)
-			(end -1.2 -1.2)
+			(end 3.2 1.2)
 			(stroke
 				(width 0.05)
@@
 		(fp_line
 			(start -1.2 1.2)
-			(end 3.2 1.2)
+			(end -1.2 -1.2)
 			(stroke
 				(width 0.05)
@@
 		)
 		(fp_text user "${REFERENCE}"
-			(at 1.1 1.7 90)
+			(at 1.1 1.7 0)
 			(layer "F.Fab")
 			(effects
@@
 		)
 		(pad "1" thru_hole circle
-			(at 0 0 90)
+			(at 0 0 180)
 			(size 1.4 1.4)
 			(drill 0.7)
@@
 		)
 		(pad "1" thru_hole circle
-			(at 2 0 90)
+			(at 2 0 180)
 			(size 1.4 1.4)
 			(drill 0.7)
@@
 	(footprint "LOGO"
 		(layer "F.Cu")
-		(at 114 62.55 -90)
+		(at 112.65 70.45 -90)
 		(property "Reference" "G***"
 			(at 0 0 90)
@@
 	(footprint "TestPoint:TestPoint_Bridge_Pitch2.0mm_Drill0.7mm"
 		(layer "F.Cu")
-		(at 112.9 70.7 90)
+		(at 116.3 70.95 90)
 		(descr "wire loop as test point, pitch 2.0mm, hole diameter 0.7mm, wire diameter 0.5mm")
 		(tags "test point wire loop")
@@
 	)
 	(via
-		(at 118.25 63.5)
+		(at 120.65 64.7)
 		(size 0.5)
 		(drill 0.3)

Commit message: modif V2 PCB
Connections:
- U1 pad 22: TX3 -> RX3
- U1 pad 24: RX3 -> TX3
Routing:
- net TX3: track 35.2 -> 27.9 mm
- net GND: vias 111 -> 113
Changed lines of the file:
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@@
 			(layers "F.Cu" "F.Mask" "F.Paste")
 			(roundrect_rratio 0.25)
-			(net 29 "TX3")
+			(net 40 "RX3")
 			(pinfunction "PB10")
 			(pintype "bidirectional")
@@
 			(layers "F.Cu" "F.Mask" "F.Paste")
 			(roundrect_rratio 0.25)
-			(net 40 "RX3")
+			(net 29 "TX3")
 			(pinfunction "PB11")
 			(pintype "bidirectional")
@@
 	)
 	(via
+		(at 123.6 96.55)
+		(size 0.5)
+		(drill 0.3)
+		(layers "F.Cu" "B.Cu")
+		(free yes)
+		(net 3)
+	)
+	(via
 		(at 154 65)
 		(size 0.5)
@@
 	)
 	(via
+		(at 129.85 93.2)
+		(size 0.5)
+		(drill 0.3)
+		(layers "F.Cu" "B.Cu")
+		(free yes)
+		(net 3)
+	)
+	(via
 		(at 125.975 87.35)
 		(size 0.5)
@@
 	)
 	(segment
-		(start 130.65 74.3975)
-		(end 130.65 75.127)
-		(width 0.2)
-		(layer "F.Cu")
-		(net 29)
-	)
-	(segment
-		(start 131.374 90.6089)
-		(end 123.9339 98.049)
-		(width 0.2)
-		(layer "F.Cu")
-		(net 29)
-	)
-	(segment
-		(start 121.479 99.67676)
-		(end 122.15324 100.351)
-		(width 0.2)
-		(layer "F.Cu")
-		(net 29)
-	)
-	(segment
-		(start 121.479 98.707479)
-		(end 121.479 99.67676)
-		(width 0.2)
-		(layer "F.Cu")
-		(net 29)
-	)
-	(segment
-		(start 130.659 75.517521)
-		(end 131.374 76.232521)
-		(width 0.2)
-		(layer "F.Cu")
-		(net 29)
-	)
-	(segment
-		(start 122.137479 98.049)
-		(end 121.479 98.707479)
-		(width 0.2)
-		(layer "F.Cu")
-		(net 29)
-	)
-	(segment
-		(start 122.15324 100.351)
-		(end 124.019 100.351)
-		(width 0.2)
-		(layer "F.Cu")
-		(net 29)
-	)
-	(segment
-		(start 131.374 76.232521)
-		(end 131.374 90.6089)
+		(start 131.775 79.175057)
+		(end 132.2 78.750057)
 		(width 0.2)
 		(layer "F.Cu")
@@
 	)
 	(segment
-		(start 130.659 75.136)
-		(end 130.659 75.517521)
+		(start 132.2 78.750057)
+		(end 132.2 74.9475)
 		(width 0.2)
 		(layer "F.Cu")
@@
 	)
 	(segment
-		(start 130.65 75.127)
-		(end 130.659 75.136)
+		(start 125.17 99.2)
+		(end 131.775 92.595)
 		(width 0.2)
 		(layer "F.Cu")
@@
 	)
 	(segment
-		(start 124.019 100.351)
-		(end 125.17 99.2)
+		(start 131.775 92.595)
+		(end 131.775 79.175057)
 		(width 0.2)
 		(layer "F.Cu")
@@
 	)
 	(segment
-		(start 123.9339 98.049)
-		(end 122.137479 98.049)
+		(start 132.2 74.9475)
+		(end 131.65 74.3975)
 		(width 0.2)
 		(layer "F.Cu")
@@
 	)
 	(segment
-		(start 132.2 74.9475)
-		(end 132.2 78.750057)
+		(start 131.374 90.776)
+		(end 131.374 76.232521)
 		(width 0.2)
 		(layer "F.Cu")
@@
 	)
 	(segment
-		(start 132.2 78.750057)
-		(end 131.775 79.175057)
+		(start 130.659 75.136)
+		(end 130.65 75.127)
 		(width 0.2)
 		(layer "F.Cu")
@@
 	)
 	(segment
-		(start 131.65 74.3975)
-		(end 132.2 74.9475)
+		(start 131.374 76.232521)
+		(end 130.659 75.517521)
 		(width 0.2)
 		(layer "F.Cu")
@@
 	)
 	(segment
-		(start 131.775 90.775)
-		(end 123.35 99.2)
+		(start 130.659 75.517521)
+		(end 130.659 75.136)
 		(width 0.2)
 		(layer "F.Cu")
@@
 	)
 	(segment
-		(start 131.775 79.175057)
-		(end 131.775 90.775)
+		(start 122.95 99.2)
+		(end 131.374 90.776)
+		(width 0.2)
+		(layer "F.Cu")
+		(net 40)
+	)
+	(segment
+		(start 122.63 99.2)
+		(end 122.95 99.2)
+		(width 0.2)
+		(layer "F.Cu")
+		(net 40)
+	)
+	(segment
+		(start 130.65 75.127)
+		(end 130.65 74.3975)
 		(width 0.2)
 		(layer "F.Cu")
