File: Hardware/KiCad V2/ChaSouRo/ChaSouRo 2.kicad_pcb (KiCad board)
At the start: 4 copper layers, 57 x 54 mm, 96 parts, among them IC1 ADXL343BCCZ-RL, IC2 ZXBM5210-SP-13, IC3 MP1475DJ-LF-P, IC4 ZXBM5210-SP-13, IC5 BU33SD5WG-TR, J1 LiDAR, J10 Motor_R, J11 BATT + ON/OFF, J12 Buzz, J2 OLED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

Commit message: maj hardware v2
Routing:
- net SDA3: track 121.0 -> 120.2 mm
Changed lines of the file:
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@@
 	)
 	(segment
-		(start 134.95 52.274)
+		(start 133.1 52.274)
 		(end 139.774 52.274)
 		(width 0.2)
@@
 	)
 	(segment
-		(start 133.1 54.11116)
-		(end 133.11284 54.11116)
+		(start 152.65 90.75)
+		(end 152.701 90.801)
+		(width 0.2)
+		(layer "F.Cu")
+		(net 43)
+	)
+	(segment
+		(start 139.774 52.274)
+		(end 141 53.5)
 		(width 0.2)
 		(layer "F.Cu")
@@
 	)
 	(segment
-		(start 152.65 90.75)
-		(end 152.701 90.801)
-		(width 0.2)
-		(layer "F.Cu")
-		(net 43)
-	)
-	(segment
 		(start 129 59.69)
 		(end 129 58.21116)
@@
 	)
 	(segment
-		(start 139.774 52.274)
-		(end 141 53.5)
+		(start 128.36 60.33)
+		(end 129 59.69)
 		(width 0.2)
 		(layer "F.Cu")
@@
 		(start 152.701 90.801)
 		(end 152.65 90.801)
-		(width 0.2)
-		(layer "F.Cu")
-		(net 43)
-	)
-	(segment
-		(start 128.65 66.89)
-		(end 128.36 66.6)
 		(width 0.2)
 		(layer "F.Cu")
@@
 	)
 	(segment
-		(start 129 58.21116)
-		(end 133.1 54.11116)
+		(start 128.65 66.89)
+		(end 128.36 66.6)
 		(width 0.2)
 		(layer "F.Cu")
@@
 	)
 	(segment
-		(start 133.11284 54.11116)
-		(end 134.95 52.274)
-		(width 0.2)
-		(layer "F.Cu")
-		(net 43)
-	)
-	(segment
 		(start 128.65 67.5225)
 		(end 128.65 66.89)
@@
 	)
 	(segment
-		(start 128.36 60.33)
-		(end 129 59.69)
-		(width 0.2)
-		(layer "F.Cu")
-		(net 43)
-	)
-	(segment
-		(start 133.1 52.274)
-		(end 134.95 52.274)
+		(start 129 58.21116)
+		(end 133.1 54.11116)
 		(width 0.2)
 		(layer "F.Cu")
@@
 		(width 0.2)
 		(layer "F.Cu")
+		(net 43)
+	)
+	(segment
+		(start 133.1 54.11116)
+		(end 133.1 52.274)
+		(width 0.2)
+		(layer "F.Cu")
