File: Hardware/KiCad V2/ChaSouRo/ChaSouRo.kicad_sch (KiCad schematic)
At the start: 41 parts, among them J3 Conn_ST_STDC14, U1 STM32G431CBUx, Y1 Crystal_GND24_Small

Commit message: maj hardware v2
Parts:
- removed C1: 4.7u, Capacitor_SMD:C_0402_1005Metric, symbol Device:C_Small
- removed C10, C2, C29, C3, C36, C37, C4, C9: 0.1u, Capacitor_SMD:C_0402_1005Metric, symbol Device:C_Small
- removed C11, C12: 22p, Capacitor_SMD:C_0402_1005Metric, symbol Device:C_Small
- removed C5: 10n, Capacitor_SMD:C_0402_1005Metric, symbol Device:C_Small
- removed C6, C8: 1u, Capacitor_SMD:C_0402_1005Metric, symbol Device:C_Small
- removed C7: 22u, Capacitor_SMD:C_0603_1608Metric, symbol Device:C_Small
- removed D1: 1, LED_SMD:LED_0603_1608Metric, symbol Device:LED
- removed D2: 2, LED_SMD:LED_0603_1608Metric, symbol Device:LED
- removed J3: Conn_ST_STDC14, Connector_PinHeader_1.27mm:PinHeader_2x07_P1.27mm_Vertical_SMD, symbol Connector:Conn_ST_STDC14
- removed L1: 4.7n, Inductor_SMD:L_0402_1005Metric, symbol Device:L
- removed R1, R2: 2.7k, Resistor_SMD:R_0402_1005Metric, symbol Device:R_Small
- removed S1: NRST, ESE:430182070816, symbol Switch:SW_Push
- removed S2: USER, ESE:430182070816, symbol Switch:SW_Push
- removed TP1: TX2, symbol Connector:TestPoint
- removed TP2: GND, TestPoint:TestPoint_Bridge_Pitch2.0mm_Drill0.7mm, symbol Connector:TestPoint
- removed TP3: 3V3, TestPoint:TestPoint_Bridge_Pitch2.0mm_Drill0.7mm, symbol Connector:TestPoint
- removed TP4: FWD_L, TestPoint:TestPoint_Bridge_Pitch2.0mm_Drill0.7mm, symbol Connector:TestPoint
- removed TP5: REV_L, TestPoint:TestPoint_Bridge_Pitch2.0mm_Drill0.7mm, symbol Connector:TestPoint
- removed TP6: FWD_R, TestPoint:TestPoint_Bridge_Pitch2.0mm_Drill0.7mm, symbol Connector:TestPoint
- removed TP7: REV_R, TestPoint:TestPoint_Bridge_Pitch2.0mm_Drill0.7mm, symbol Connector:TestPoint
- removed TP8: USER2, symbol Connector:TestPoint
- removed U1: STM32G431CBUx, Package_DFN_QFN:QFN-48-1EP_7x7mm_P0.5mm_EP5.6x5.6mm, symbol MCU_ST_STM32G4:STM32G431CBUx
- removed Y1: Crystal_GND24_Small, Crystal:Crystal_SMD_3225-4Pin_3.2x2.5mm, symbol Device:Crystal_GND24_Small
Connections:
- net SCL1 renamed MCU/SCL1
- net SCL3 renamed MCU/SDA3
- net SDA1 renamed MCU/SDA1
- net SDA3 renamed MCU/SCL3
- no-connect marks 8 -> 0
Other:
- added sheet MCU (MCU.kicad_sch)
- note removed: "Pour les ADC"
- moved on the sheet: H1, H2, H3, H4, R3, R4, R5, R6
